File: bsc_ext_serial.kicad_pcb (KiCad board)
At the start: 4 copper layers, 100 x 100 mm, 176 parts, among them J1 Conn_Adr, J2 Conn_Bus, Q1 BC857BS, Q2 IRLML2244, Q3 BC857BS, Q4 IRLML2244, U1 MCP23017_SO, U2 ADM2483xRW, U3 ADM2483xRW, U4 ADM2483xRW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

Commit message: modify J2 position
Parts:
- moved R47 18.6 mm to (50.5, 99.8), turned to 0 degrees
- moved R6 17.4 mm to (35.7, 95.2), turned to -90 degrees
- moved R5 17.3 mm to (33.8, 95.2), turned to -90 degrees
- moved R48 14.8 mm to (50.6, 96.4), turned to 0 degrees
- moved D3 14.3 mm to (35.7, 91.9), turned to -90 degrees
- moved D2 14.2 mm to (33.8, 91.9), turned to -90 degrees
- moved R4 12.9 mm to (38.0, 95.2), turned to -90 degrees
- moved D1 8.22 mm to (38.0, 91.8), turned to 90 degrees
- moved D14 5.25 mm to (63.4, 75.7)
- moved D16 5.25 mm to (67.2, 75.7)
- moved D19 5.25 mm to (73.1, 75.7)
- moved D4 5.25 mm to (41.3, 75.7)
- moved D5 5.25 mm to (43.1, 75.7)
- moved D7 5.25 mm to (46.9, 75.7)
- moved R10 5.25 mm to (46.9, 78.9)
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Routing:
- net /U3RX_EN: track 63.7 -> 55.7 mm, vias 3 -> 2
- net /U2TX_EN: track 65.6 -> 58.5 mm, vias 2 -> 4
- net +3V3: track 85.8 -> 79.8 mm, vias 25 -> 28
- net /U_TX: track 226.2 -> 231.5 mm, vias 14 -> 13
- net /U2RX_EN: track 57.8 -> 52.9 mm
- net /SCL: track 26.9 -> 30.7 mm
- net /U_RX: track 226.8 -> 230.5 mm, vias 3 -> 2
- net /SDA: track 26.9 -> 30.2 mm
- net /U1TX_EN: track 56.4 -> 53.2 mm
- net /U4TX_EN: track 68.6 -> 71.3 mm
- net +5V: track 310.1 -> 307.4 mm
- net /U8RX_EN: track 59.5 -> 62.0 mm
- net /U1RX_EN: track 54.1 -> 51.7 mm, vias 3 -> 2
- net /U6RX_EN: track 91.0 -> 89.7 mm, vias 2 -> 3
- net /U6TX_EN: track 92.4 -> 91.1 mm
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Other:
- board text added: "1 |"
- board text added: "2 |"
- board text added: "3 |"
- board text added: "4"
- board text added: "5 |"
- board text added: "6 |"
- board text added: "7 |"
- board text added: "8"
- board text added: "Rx"
- board text added: "Tx"
- board text added: "Tx/Rx EN"
- board text removed: "2 3 4 5 6 7 8"
- board text removed: "EN TxRx"
- board text removed: "Tx Rx"
